Commit message: Change global frame, fix caster wheel

File: src/model_robot/urdf/diff_offset_robot.urdf (robot description, URDF)
Before this commit: robot diff_offset_robot, 6 links, 5 joints
Joints:
- joint caster_wheel_joint: origin xyz=0.23725 0 -0.025 rpy=-3.1416 0 -0.53405 -> xyz=0.125 0 -0.005 rpy=-3.1416 0 -0.53405
- joint left_wheel_joint: origin xyz=0 0.13 0 rpy=-1.5708 0.05745 0 -> xyz=-0.11225 0.13 0.02 rpy=-1.5708 0.05745 0
- joint lidar_joint: origin xyz=0.29225 0 0.03 rpy=0 0 0 -> xyz=0.18 0 0.05 rpy=0 0 0
- joint right_wheel_joint: origin xyz=0 -0.13 0 rpy=-1.5708 0 0 -> xyz=-0.11225 -0.13 0.02 rpy=-1.5708 0 0
- joint top_base_joint: origin xyz=0.11225 0 0.03 rpy=0 0 0 -> xyz=0 0 0.05 rpy=0 0 0
