Commit message: Change Robot

File: install/model_robot/share/model_robot/urdf/diff_offset_robot.urdf (robot description, URDF)
Before this commit: robot diff_offset_robot, 6 links, 5 joints
Links:
- added link body_wheel_link, mass 0.038337; collision mesh filename=package://model_robot/meshes/body_wheel_link.STL; visual mesh filename=package://model_robot/meshes/body_wheel_link.STL
- link base_link: mass 7.674 -> 6.20721211987107
- link caster_wheel_link: mass 0.056549 -> 0.01313
- link left_wheel_link: mass 0.5702 -> 0.37174
- link right_wheel_link: mass 0.5702 -> 0.37174
Joints:
- added joint body_wheel_joint: type continuous, parent base_link, child body_wheel_link, origin xyz=0.125 0 0.004 rpy=3.1416 0 0.0019842, axis 0 0 1, limit effort=100 velocity=100
- joint caster_wheel_joint: axis 0 0 0 -> 0 0 1; limit (none) -> effort=100 velocity=100; origin xyz=0.23725 0 -0.025 rpy=-3.1416 0 -0.53405 -> xyz=0.016 0 0.023 rpy=1.5708 -0.40647 0; parent base_link -> body_wheel_link; type fixed -> continuous
- joint left_wheel_joint: origin xyz=0 0.13 0 rpy=-1.5708 0.05745 0 -> xyz=-0.11225 0.13 0.02 rpy=-1.5708 0.05745 0
- joint lidar_joint: origin xyz=0.29225 0 0.03 rpy=0 0 0 -> xyz=0.18 0 0.05 rpy=0 0 0
- joint right_wheel_joint: origin xyz=0 -0.13 0 rpy=-1.5708 0 0 -> xyz=-0.11225 -0.13 0.02 rpy=-1.5708 0 0
- joint top_base_joint: origin xyz=0.11225 0 0.03 rpy=0 0 0 -> xyz=0 0 0.05 rpy=0 0 0

File: src/model_robot/urdf/diff_offset_robot.urdf (robot description, URDF)
Before this commit: robot diff_offset_robot, 6 links, 5 joints
Links:
- added link body_wheel_link, mass 0.038337; collision mesh filename=package://model_robot/meshes/body_wheel_link.STL; visual mesh filename=package://model_robot/meshes/body_wheel_link.STL
- link base_link: mass 7.674 -> 6.20721211987107
- link caster_wheel_link: mass 0.056549 -> 0.01313
- link left_wheel_link: mass 0.5702 -> 0.37174
- link right_wheel_link: mass 0.5702 -> 0.37174
Joints:
- added joint body_wheel_joint: type continuous, parent base_link, child body_wheel_link, origin xyz=0.125 0 0.004 rpy=3.1416 0 0.0019842, axis 0 0 1, limit effort=100 velocity=100
- joint caster_wheel_joint: axis 0 0 0 -> 0 0 1; limit (none) -> effort=100 velocity=100; origin xyz=0.125 0 -0.005 rpy=-3.1416 0 -0.53405 -> xyz=0.016 0 0.023 rpy=1.5708 -0.40647 0; parent base_link -> body_wheel_link; type fixed -> continuous

Commit message: change frames

File: install/model_robot/share/model_robot/urdf/diff_offset_robot.urdf (robot description, URDF)
Before this commit: robot diff_offset_robot, 7 links, 6 joints
Joints:
- joint left_wheel_joint: origin xyz=-0.11225 0.13 0.02 rpy=-1.5708 0.05745 0 -> xyz=-0.11225 0.13 0.02 rpy=0 0 1.5708

Commit message: Successful robot simulation

File: install/model_robot/share/model_robot/urdf/diff_offset_robot.urdf (robot description, URDF)
Before this commit: robot diff_offset_robot, 7 links, 6 joints
Links:
- link base_link: mass 6.20721211987107 -> 16.759
- link body_wheel_link: mass 0.038337 -> 0.045198
- link caster_wheel_link: mass 0.01313 -> 0.015177
- link lidar_link: mass 0.15681 -> 0.19445
- link top_base_link: mass 6.1261 -> 16.54
Joints:
- joint body_wheel_joint: origin xyz=0.125 0 0.004 rpy=3.1416 0 0.0019842 -> xyz=0.125 0 -0.016 rpy=-3.1416 0 0
- joint caster_wheel_joint: origin xyz=0.016 0 0.023 rpy=1.5708 -0.40647 0 -> xyz=0.016 0 0.023 rpy=1.5708 0 0
- joint left_wheel_joint: origin xyz=-0.11225 0.13 0.02 rpy=0 0 1.5708 -> xyz=-0.11225 0.13 0 rpy=1.5708 0.57871 3.1416
- joint lidar_joint: origin xyz=0.18 0 0.05 rpy=0 0 0 -> xyz=0.18 0 0.03 rpy=0 0 0
- joint right_wheel_joint: origin xyz=-0.11225 -0.13 0.02 rpy=-1.5708 0 0 -> xyz=-0.11225 -0.13 0 rpy=-1.5708 -0.061252 0
- joint top_base_joint: limit lower=0 upper=6.2832 effort=100 velocity=100 -> lower=0 upper=6.28 effort=0 velocity=0; origin xyz=0 0 0.05 rpy=0 0 0 -> xyz=0 0 0.03 rpy=0 0 0

File: src/model_robot/urdf/diff_offset_robot.urdf (robot description, URDF)
Before this commit: robot diff_offset_robot, 7 links, 6 joints
Links:
- link base_link: mass 6.20721211987107 -> 16.759
- link body_wheel_link: mass 0.038337 -> 0.045198
- link caster_wheel_link: mass 0.01313 -> 0.015177
- link lidar_link: mass 0.15681 -> 0.19445
- link top_base_link: mass 6.1261 -> 16.54
Joints:
- joint body_wheel_joint: origin xyz=0.125 0 0.004 rpy=3.1416 0 0.0019842 -> xyz=0.125 0 -0.016 rpy=-3.1416 0 0
- joint caster_wheel_joint: origin xyz=0.016 0 0.023 rpy=1.5708 -0.40647 0 -> xyz=0.016 0 0.023 rpy=1.5708 0 0
- joint left_wheel_joint: origin xyz=-0.11225 0.13 0.02 rpy=-1.5708 0.05745 0 -> xyz=-0.11225 0.13 0 rpy=1.5708 0.57871 3.1416
- joint lidar_joint: origin xyz=0.18 0 0.05 rpy=0 0 0 -> xyz=0.18 0 0.03 rpy=0 0 0
- joint right_wheel_joint: origin xyz=-0.11225 -0.13 0.02 rpy=-1.5708 0 0 -> xyz=-0.11225 -0.13 0 rpy=-1.5708 -0.061252 0
- joint top_base_joint: limit lower=0 upper=6.2832 effort=100 velocity=100 -> lower=0 upper=6.28 effort=0 velocity=0; origin xyz=0 0 0.05 rpy=0 0 0 -> xyz=0 0 0.03 rpy=0 0 0

Commit message: Change robot and Implementacion Kinematics node

File: install/model_robot/share/model_robot/urdf/diff_offset_robot.urdf (robot description, URDF)
Before this commit: robot diff_offset_robot, 7 links, 6 joints
Links:
- removed link body_wheel_link
- removed link caster_wheel_link
- link base_link: mass 16.759 -> 7.7306
- link lidar_link: mass 0.19445 -> 0.15681
- link top_base_link: mass 16.54 -> 6.1261
Joints:
- removed joint body_wheel_joint
- removed joint caster_wheel_joint
- joint left_wheel_joint: origin xyz=-0.11225 0.13 0 rpy=1.5708 0.57871 3.1416 -> xyz=-0.11225 0.13 0 rpy=-1.5708 0.05745 0
- joint right_wheel_joint: origin xyz=-0.11225 -0.13 0 rpy=-1.5708 -0.061252 0 -> xyz=-0.11225 -0.13 0 rpy=-1.5708 0 0
- joint top_base_joint: limit lower=0 upper=6.28 effort=0 velocity=0 -> lower=0 upper=6.2832 effort=100 velocity=100
