Commit message: Teleop node created

File: install/model_robot/share/model_robot/urdf/diff_offset_robot.urdf.xacro (robot description, xacro)
@@ -95,6 +95,6 @@
       xyz="0 0 1" />
     <limit
-      effort="100"
-      velocity="100" />
+      effort="10"
+      velocity="20" />
     <dynamics
       damping="0.1"
@@ -128,5 +128,5 @@
         name="">
         <color
-          rgba="0.019608 0 0 1" />
+          rgba="0.019608 0 0 -1" />
       </material>
     </visual>
@@ -154,6 +154,6 @@
       xyz="0 0 1" />
     <limit
-      effort="100"
-      velocity="100" />
+      effort="10"
+      velocity="20" />
     <dynamics
       damping="0.1"
@@ -215,6 +215,6 @@
       lower="0"
       upper="6.2832"
-      effort="100"
-      velocity="100" />
+      effort="10"
+      velocity="20" />
     <dynamics
       damping="0.1"
@@ -276,4 +276,7 @@
       effort="100"
       velocity="100" />
+    <dynamics
+      damping="0.1"
+      friction="0.1" />
   </joint>
   <ros2_control name="diff_offset_robot_control" type="system">

Commit message: Fixed Maths, fixed publication of joint states, adds rviz configuration and data_logger file allows to create charts

File: install/model_robot/share/model_robot/urdf/diff_offset_robot.urdf.xacro (robot description, xacro)
@@ -6,15 +6,15 @@
     <inertial>
       <origin
-        xyz="0.027195 -1.382E-07 1.4192E-05"
-        rpy="0 0 0" />
-      <mass
-        value="7.7306" />
-      <inertia
-        ixx="0.08923"
-        ixy="-1.6849E-17"
-        ixz="-0.00013721"
-        iyy="0.12656"
-        iyz="-1.6354E-19"
-        izz="0.21251" />
+        xyz="0.0077925 1.382E-07 0.0044813"
+        rpy="0 0 0" />
+      <mass
+        value="16.766" />
+      <inertia
+        ixx="0.17714"
+        ixy="-2.225E-17"
+        ixz="-0.0072719"
+        iyy="0.29215"
+        iyz="1.8084E-15"
+        izz="0.4637" />
     </inertial>
     <visual>
@@ -29,5 +29,5 @@
         name="">
         <color
-          rgba="0.79216 0.81961 0.93333 1" />
+          rgba="0.86667 0.9098 1 1" />
       </material>
     </visual>
@@ -46,5 +46,5 @@
     <inertial>
       <origin
-        xyz="-2.2204E-16 -3.2613E-16 0.04781"
+        xyz="2.2204E-16 -7.7716E-16 0.04781"
         rpy="0 0 0" />
       <mass
@@ -52,8 +52,8 @@
       <inertia
         ixx="0.00039822"
-        ixy="-1.2163E-18"
-        ixz="-3.573E-19"
+        ixy="6.9118E-19"
+        ixz="4.4212E-19"
         iyy="0.00039822"
-        iyz="-9.9603E-19"
+        iyz="-2.2832E-18"
         izz="0.00057276" />
     </inertial>
@@ -87,5 +87,5 @@
     <origin
       xyz="-0.11225 0.13 0"
-      rpy="-1.5708 0.05745 0" />
+      rpy="1.5708 0.57871 3.1416" />
     <parent
       link="base_link" />
@@ -95,5 +95,5 @@
       xyz="0 0 1" />
     <limit
-      effort="10"
+      effort="50"
       velocity="20" />
     <dynamics
@@ -105,5 +105,5 @@
     <inertial>
       <origin
-        xyz="4.4409E-16 2.3245E-16 -0.04781"
+        xyz="6.6613E-16 -2.2204E-16 -0.04781"
         rpy="0 0 0" />
       <mass
@@ -111,8 +111,8 @@
       <inertia
         ixx="0.00039822"
-        ixy="1.5059E-18"
-        ixz="-3.6035E-19"
+        ixy="-2.7444E-19"
+        ixz="3.7384E-19"
         iyy="0.00039822"
-        iyz="-6.9788E-19"
+        iyz="3.2089E-19"
         izz="0.00057276" />
     </inertial>
@@ -128,5 +128,5 @@
         name="">
         <color
-          rgba="0.019608 0 0 -1" />
+          rgba="0.019608 0 0 1" />
       </material>
     </visual>
@@ -146,5 +146,5 @@
     <origin
       xyz="-0.11225 -0.13 0"
-      rpy="-1.5708 0 0" />
+      rpy="-1.5708 -0.061252 0" />
     <parent
       link="base_link" />
@@ -154,5 +154,5 @@
       xyz="0 0 1" />
     <limit
-      effort="10"
+      effort="50"
       velocity="20" />
     <dynamics
@@ -161,58 +161,56 @@
   </joint>
   <link
-    name="top_base_link">
-    <inertial>
-      <origin
-        xyz="4.4409E-16 -1.5959E-16 0.043846"
-        rpy="0 0 0" />
-      <mass
-        value="6.1261" />
-      <inertia
-        ixx="0.092849"
-        ixy="2.2239E-18"
-        ixz="-1.0728E-18"
-        iyy="0.092849"
-        iyz="-4.5642E-20"
-        izz="0.18437" />
-    </inertial>
-    <visual>
-      <origin
-        xyz="0 0 0"
-        rpy="0 0 0" />
-      <geometry>
-        <mesh
-          filename="package://model_robot/meshes/top_base_link.STL" />
-      </geometry>
-      <material
-        name="">
-        <color
-          rgba="0.48235 0.61176 1 1" />
-      </material>
-    </visual>
-    <collision>
-      <origin
-        xyz="0 0 0"
-        rpy="0 0 0" />
-      <geometry>
-        <mesh
-          filename="package://model_robot/meshes/top_base_link.STL" />
-      </geometry>
-    </collision>
-  </link>
-  <joint
-    name="top_base_joint"
-    type="revolute">
-    <origin
-      xyz="0 0 0.03"
+    name="lidar_link">
+    <inertial>
+      <origin
+        xyz="-2.22044604925031E-16 0 0.00998372049732055"
+        rpy="0 0 0" />
+      <mass
+        value="0.194447333272832" />
+      <inertia
+        ixx="0.000127792042048439"
+        ixy="-3.36102673470719E-21"
+        ixz="1.19867346730935E-18"
+        iyy="0.000127792042048439"
+        iyz="1.19874708938594E-18"
+        izz="0.000242659502252698" />
+    </inertial>
+    <visual>
+      <origin
+        xyz="0 0 0"
+        rpy="0 0 0" />
+      <geometry>
+        <mesh
+          filename="package://model_robot/meshes/lidar_link.STL" />
+      </geometry>
+      <material
+        name="">
+        <color
+          rgba="0.698039215686274 0.698039215686274 0.698039215686274 1" />
+      </material>
+    </visual>
+    <collision>
+      <origin
+        xyz="0 0 0"
+        rpy="0 0 0" />
+      <geometry>
+        <mesh
+          filename="package://model_robot/meshes/lidar_link.STL" />
+      </geometry>
+    </collision>
+  </link>
+  <joint
+    name="lidar_joint"
+    type="continuous">
+    <origin
+      xyz="0.18 0 0.03"
       rpy="0 0 0" />
     <parent
       link="base_link" />
     <child
-      link="top_base_link" />
+      link="lidar_link" />
     <axis
       xyz="0 0 1" />
     <limit
-      lower="0"
-      upper="6.2832"
       effort="10"
       velocity="20" />
@@ -222,61 +220,177 @@
   </joint>
   <link
-    name="lidar_link">
-    <inertial>
-      <origin
-        xyz="0 -6.9389E-18 0.0099837"
-        rpy="0 0 0" />
-      <mass
-        value="0.15681" />
-      <inertia
-        ixx="0.00010306"
-        ixy="-6.0185E-36"
-        ixz="-2.3099E-21"
-        iyy="0.00010306"
-        iyz="5.8547E-22"
-        izz="0.00019569" />
-    </inertial>
-    <visual>
-      <origin
-        xyz="0 0 0"
-        rpy="0 0 0" />
-      <geometry>
-        <mesh
-          filename="package://model_robot/meshes/lidar_link.STL" />
-      </geometry>
-      <material
-        name="">
-        <color
-          rgba="0.94118 0.16863 0 1" />
-      </material>
-    </visual>
-    <collision>
-      <origin
-        xyz="0 0 0"
-        rpy="0 0 0" />
-      <geometry>
-        <mesh
-          filename="package://model_robot/meshes/lidar_link.STL" />
-      </geometry>
-    </collision>
-  </link>
-  <joint
-    name="lidar_joint"
-    type="continuous">
-    <origin
-      xyz="0.18 0 0.03"
+    name="top_base_link">
+    <inertial>
+      <origin
+        xyz="8.8818E-16 8.8818E-16 0.043846"
+        rpy="0 0 0" />
+      <mass
+        value="16.54" />
+      <inertia
+        ixx="0.25069"
+        ixy="4.8639E-18"
+        ixz="2.5866E-15"
+        iyy="0.25069"
+        iyz="2.5916E-15"
+        izz="0.4978" />
+    </inertial>
+    <visual>
+      <origin
+        xyz="0 0 0"
+        rpy="0 0 0" />
+      <geometry>
+        <mesh
+          filename="package://model_robot/meshes/top_base_link.STL" />
+      </geometry>
+      <material
+        name="">
+        <color
+          rgba="0.86667 0.9098 1 1" />
+      </material>
+    </visual>
+    <collision>
+      <origin
+        xyz="0 0 0"
+        rpy="0 0 0" />
+      <geometry>
+        <mesh
+          filename="package://model_robot/meshes/top_base_link.STL" />
+      </geometry>
+    </collision>
+  </link>
+  <joint
+    name="top_base_joint"
+    type="revolute">
+    <origin
+      xyz="0 0 0.03"
       rpy="0 0 0" />
     <parent
       link="base_link" />
     <child
-      link="lidar_link" />
+      link="top_base_link" />
     <axis
       xyz="0 0 1" />
     <limit
-      effort="100"
-      velocity="100" />
+      lower="0"
+      upper="6.28"
+      effort="10"
+      velocity="20" />
     <dynamics
       damping="0.1"
       friction="0.1" />
+  </joint>
+  <link
+    name="body_wheel_link">
+    <inertial>
+      <origin
+        xyz="0.0012182 3.9726E-05 0.012909"
+        rpy="0 0 0" />
+      <mass
+        value="0.067446" />
+      <inertia
+        ixx="1.7013E-05"
+        ixy="1.4706E-07"
+        ixz="1.1675E-07"
+        iyy="1.2508E-05"
+        iyz="3.8073E-09"
+        izz="1.9263E-05" />
+    </inertial>
+    <visual>
+      <origin
+        xyz="0 0 0"
+        rpy="0 0 0" />
+      <geometry>
+        <mesh
+          filename="package://model_robot/meshes/body_wheel_link.STL" />
+      </geometry>
+      <material
+        name="">
+        <color
+          rgba="0.77647 0.75686 0.73725 1" />
+      </material>
+    </visual>
+    <collision>
+      <origin
+        xyz="0 0 0"
+        rpy="0 0 0" />
+      <geometry>
+        <mesh
+          filename="package://model_robot/meshes/body_wheel_link.STL" />
+      </geometry>
+    </collision>
+  </link>
+  <joint
+    name="body_wheel_joint"
+    type="continuous">
+    <origin
+      xyz="0.18 0 -0.015"
+      rpy="3.1416 0 0" />
+    <parent
+      link="base_link" />
+    <child
+      link="body_wheel_link" />
+    <axis
+      xyz="0 0 1" />
+    <limit
+      effort="10"
+      velocity="20" />
+    <dynamics
+      damping="0.01"/>
+  </joint>
+  <link
+    name="caster_wheel_link">
+    <inertial>
+      <origin
+        xyz="-2.2204E-16 2.2204E-16 0"
+        rpy="0 0 0" />
+      <mass
+        value="0.034498" />
+      <inertia
+        ixx="5.4969E-06"
+        ixy="-6.3793E-23"
+        ixz="2.4265E-08"
+        iyy="5.4961E-06"
+        iyz="-1.9562E-21"
+        izz="6.2402E-06" />
+    </inertial>
+    <visual>
+      <origin
+        xyz="0 0 0"
+        rpy="0 0 0" />
+      <geometry>
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
Commit message: SIntonizacion PID para ruedas

File: install/model_robot/share/model_robot/urdf/diff_offset_robot.urdf.xacro (robot description, xacro)
@@ -259,5 +259,13 @@
     </collision>
   </link>
-  <joint
+  <joint name="top_base_joint" type="continuous">
+    <origin xyz="0 0 0.03" rpy="0 0 0" />
+    <parent link="base_link" />
+    <child link="top_base_link" />
+    <axis xyz="0 0 1" />
+    <limit effort="1000.0" velocity="20.0" />
+    <dynamics damping="0.1" friction="0.1" />
+  </joint>
+  <!-- <joint
     name="top_base_joint"
     type="revolute">
@@ -279,5 +287,5 @@
       damping="0.1"
       friction="0.1" />
-  </joint>
+  </joint> -->
   <link
     name="body_wheel_link">
@@ -400,16 +408,22 @@
     <joint name="left_wheel_joint">
       <command_interface name="velocity"/>
+      <command_interface name="effort"/>
       <state_interface name="position"/>
       <state_interface name="velocity"/>
+      <state_interface name="effort"/>
     </joint>
     <joint name="right_wheel_joint">
       <command_interface name="velocity"/>
+      <command_interface name="effort"/>
       <state_interface name="position"/>
       <state_interface name="velocity"/>
+      <state_interface name="effort"/>
     </joint>
     <joint name="top_base_joint">
       <command_interface name="velocity"/>
+      <command_interface name="effort"/>
       <state_interface name="position"/>
       <state_interface name="velocity"/>
+      <state_interface name="effort"/>
     </joint>
   </ros2_control>

Commit message: Implementacion SLAM

File: install/model_robot/share/model_robot/urdf/diff_offset_robot.urdf.xacro (robot description, xacro)
@@ -468,5 +468,5 @@
         </scan>
         <range>
-          <min>0.15</min>
+          <min>0.45</min>
           <max>12.0</max>
           <resolution>0.01</resolution>

File: src/model_robot/urdf/diff_offset_robot.urdf.xacro (robot description, xacro)
@@ -259,13 +259,5 @@
     </collision>
   </link>
-  <joint name="top_base_joint" type="continuous">
-    <origin xyz="0 0 0.03" rpy="0 0 0" />
-    <parent link="base_link" />
-    <child link="top_base_link" />
-    <axis xyz="0 0 1" />
-    <limit effort="1000.0" velocity="20.0" />
-    <dynamics damping="0.1" friction="0.1" />
-  </joint>
-  <!-- <joint
+  <joint
     name="top_base_joint"
     type="revolute">
@@ -287,5 +279,5 @@
       damping="0.1"
       friction="0.1" />
-  </joint> -->
+  </joint>
   <link
     name="body_wheel_link">
@@ -468,5 +460,5 @@
         </scan>
         <range>
-          <min>0.15</min>
+          <min>0.45</min>
           <max>12.0</max>
           <resolution>0.01</resolution>

Commit message: Slam fixed, lidar

File: install/model_robot/share/model_robot/urdf/diff_offset_robot.urdf.xacro (robot description, xacro)
@@ -202,5 +202,5 @@
   <joint
     name="lidar_joint"
-    type="continuous">
+    type="fixed">
     <origin
       xyz="0.18 0 0.03"
@@ -259,13 +259,5 @@
     </collision>
   </link>
-  <joint name="top_base_joint" type="continuous">
-    <origin xyz="0 0 0.03" rpy="0 0 0" />
-    <parent link="base_link" />
-    <child link="top_base_link" />
-    <axis xyz="0 0 1" />
-    <limit effort="1000.0" velocity="20.0" />
-    <dynamics damping="0.1" friction="0.1" />
-  </joint>
-  <!-- <joint
+  <joint
     name="top_base_joint"
     type="revolute">
@@ -287,5 +279,5 @@
       damping="0.1"
       friction="0.1" />
-  </joint> -->
+  </joint>
   <link
     name="body_wheel_link">
@@ -431,5 +423,4 @@
     <plugin name="gazebo_lidar_joint_state" filename="libgazebo_ros_joint_state_publisher.so">
       <update_rate>100</update_rate>
-      <joint_name>lidar_joint</joint_name>
       <joint_name>body_wheel_joint</joint_name>
       <joint_name>caster_wheel_joint</joint_name>

File: src/model_robot/urdf/diff_offset_robot.urdf.xacro (robot description, xacro)
@@ -202,5 +202,5 @@
   <joint
     name="lidar_joint"
-    type="continuous">
+    type="fixed">
     <origin
       xyz="0.18 0 0.03"
@@ -423,5 +423,4 @@
     <plugin name="gazebo_lidar_joint_state" filename="libgazebo_ros_joint_state_publisher.so">
       <update_rate>100</update_rate>
-      <joint_name>lidar_joint</joint_name>
       <joint_name>body_wheel_joint</joint_name>
       <joint_name>caster_wheel_joint</joint_name>
